Commit message: maybe floor fix

File: src/sec_bot/description/camera.xacro (robot description, xacro)
@@ -1,8 +1,12 @@
 <?xml version="1.0"?>
 <robot xmlns:xacro="http://www.ros.org/wiki/xacro" >
+    <material name="camera_red">
+      <color rgba="1 0 0 1"/>
+    </material>
+    <!-- Left Camera -->
     <joint name="camera_joint" type="fixed">
         <parent link="chassis"/>
         <child link="camera_link"/>
-        <origin xyz="0.32 0.1400242 0.25" rpy="0 0 0"/>
+        <origin xyz="0.12 0.12 0.25" rpy="0 0 0"/>
     </joint>
     <link name="camera_link">
@@ -11,6 +15,15 @@
                 <box size="0.010 0.03 0.03"/>
             </geometry>
-            <material name="red"/>
+            <material name="camera_red"/>
         </visual>
+        <collision>
+            <geometry>
+                <box size="0.010 0.03 0.03"/>
+            </geometry>
+        </collision>
+        <inertial>
+            <mass value="0.05"/>
+            <inertia ixx="0.0001" ixy="0" ixz="0" iyy="0.0001" iyz="0" izz="0.0001"/>
+        </inertial>
     </link>
     <joint name="camera_optical_joint" type="fixed">
@@ -20,31 +33,9 @@
     </joint>
     <link name="camera_link_optical"></link>
-    <gazebo reference="camera_link">
-        <material>Gazebo/Red</material>
-        <sensor name="camera" type="camera">
-            <pose> 0 0 0 0 0 0 </pose>
-            <visualize>true</visualize>
-            <update_rate>10</update_rate>
-            <camera>
-                <horizontal_fov>1.089</horizontal_fov>
-                <image>
-                    <format>R8G8B8</format>
-                    <width>640</width>
-                    <height>480</height>
-                </image>
-                <clip>
-                    <near>0.05</near>
-                    <far>8.0</far>
-                </clip>
-            </camera>
-            <plugin name="camera_controller" filename="libgazebo_ros_camera.so">
-                <frame_name>camera_link_optical</frame_name>
-            </plugin>
-        </sensor>
-    </gazebo>
+    <!-- Right Camera -->
     <joint name="camera2_joint" type="fixed">
         <parent link="chassis"/>
         <child link="camera2_link"/>
-        <origin xyz="0.32 -0.1400242 0.25" rpy="0 0 0"/>
+        <origin xyz="0.12 -0.12 0.25" rpy="0 0 0"/>
     </joint>
     <link name="camera2_link">
@@ -53,6 +44,15 @@
                 <box size="0.010 0.03 0.03"/>
             </geometry>
-            <material name="red"/>
+            <material name="camera_red"/>
         </visual>
+        <collision>
+            <geometry>
+                <box size="0.010 0.03 0.03"/>
+            </geometry>
+        </collision>
+        <inertial>
+            <mass value="0.05"/>
+            <inertia ixx="0.0001" ixy="0" ixz="0" iyy="0.0001" iyz="0" izz="0.0001"/>
+        </inertial>
     </link>
     <joint name="camera2_optical_joint" type="fixed">
@@ -62,26 +62,3 @@
     </joint>
     <link name="camera2_link_optical"></link>
-    <gazebo reference="camera2_link">
-        <material>Gazebo/Red</material>
-        <sensor name="camera2" type="camera">
-            <pose> 0 0 0 0 0 0 </pose>
-            <visualize>true</visualize>
-            <update_rate>10</update_rate>
-            <camera>
-                <horizontal_fov>1.089</horizontal_fov>
-                <image>
-                    <format>R8G8B8</format>
-                    <width>640</width>
-                    <height>480</height>
-                </image>
-                <clip>
-                    <near>0.05</near>
-                    <far>8.0</far>
-                </clip>
-            </camera>
-            <plugin name="camera2_controller" filename="libgazebo_ros_camera.so">
-                <frame_name>camera2_link_optical</frame_name>
-            </plugin>
-        </sensor>
-    </gazebo>
 </robot>

File: src/sec_bot/description/gazebo_control.xacro (robot description, xacro)
@@ -1,36 +1,53 @@
 <?xml version="1.0"?>
-<robot xmlns:xacro="http://www.ros.org/wiki/xacro"  name="robot">
-  <gazebo>
-    <plugin name="diff_drive" filename="libgazebo_ros_diff_drive.so">
-      <!-- Wheel Information -->
-      <!-- 2 wheels per side -->
-      <num_wheel_pairs>2</num_wheel_pairs>
-      <!-- Left Wheels -->
-      <left_joint>
-        left_front_wheel_joint
-      </left_joint>
-      <left_joint>
-        left_back_wheel_joint
-      </left_joint>
-      <!-- Right Wheels -->
-      <right_joint>
-        right_front_wheel_joint
-      </right_joint>
-      <right_joint>
-        right_back_wheel_joint
-      </right_joint>
-      <!-- Wheel Definitions -->
-      <wheel_seperation>0.2800484</wheel_seperation>
-      <wheel_diameter>0.1651</wheel_diameter>
-      <!-- Limits -->
-      <max_wheel_torque>200</max_wheel_torque>
-      <max_wheel_acceleration>10</max_wheel_acceleration>
-      <!-- Output -->
-      <odometry_frame>odom</odometry_frame>
-      <robot_base_frame>base_link</robot_base_frame>
-      <publish_odom>true</publish_odom>
-      <publish_odom_tf>true</publish_odom_tf>
-      <publish_wheel_tf>true</publish_wheel_tf>
-    </plugin>
-  </gazebo>
+<robot xmlns:xacro="http://www.ros.org/wiki/xacro" >
+    <!-- Define PI if not already defined -->
+    <xacro:property name="PI" value="3.1415926535897931" />
+    <!-- Camera Gazebo Integration -->
+    <gazebo reference="camera_link">
+        <material>Gazebo/Red</material>
+        <sensor name="camera" type="camera">
+            <pose> 0 0 0 0 0 0 </pose>
+            <visualize>true</visualize>
+            <update_rate>10</update_rate>
+            <camera>
+                <horizontal_fov>1.089</horizontal_fov>
+                <image>
+                    <format>R8G8B8</format>
+                    <width>640</width>
+                    <height>480</height>
+                </image>
+                <clip>
+                    <near>0.05</near>
+                    <far>8.0</far>
+                </clip>
+            </camera>
+            <plugin name="camera_controller" filename="libgazebo_ros_camera.so">
+                <frame_name>camera_link_optical</frame_name>
+            </plugin>
+        </sensor>
+    </gazebo>
+    <gazebo reference="camera2_link">
+        <material>Gazebo/Red</material>
+        <sensor name="camera2" type="camera">
+            <pose> 0 0 0 0 0 0 </pose>
+            <visualize>true</visualize>
+            <update_rate>10</update_rate>
+            <camera>
+                <horizontal_fov>1.089</horizontal_fov>
+                <image>
+                    <format>R8G8B8</format>
+                    <width>640</width>
+                    <height>480</height>
+                </image>
+                <clip>
+                    <near>0.05</near>
+                    <far>8.0</far>
+                </clip>
+            </camera>
+            <plugin name="camera2_controller" filename="libgazebo_ros_camera.so">
+                <frame_name>camera2_link_optical</frame_name>
+            </plugin>
+        </sensor>
+    </gazebo>
+    <!-- Add other Gazebo control plugins here -->
 </robot>

File: src/sec_bot/description/inertial_macros.xacro (robot description, xacro)
@@ -4,5 +4,5 @@
   <xacro:macro name="inertial_box"
                params="mass:=1.0 x:=0.1 y:=0.1 z:=0.1
-                       origin_xyz:=0 0 0 origin_rpy:=0 0 0">
+                       origin_xyz:='0 0 0' origin_rpy:='0 0 0'">
     <inertial>
       <origin xyz="${origin_xyz}" rpy="${origin_rpy}"/>
@@ -18,5 +18,5 @@
   <xacro:macro name="inertial_cylinder"
                params="mass:=1.0 radius:=0.1 length:=0.1
-                       origin_xyz:=0 0 0 origin_rpy:=0 0 0">
+                       origin_xyz:='0 0 0' origin_rpy:='0 0 0'">
     <inertial>
       <origin xyz="${origin_xyz}" rpy="${origin_rpy}"/>
@@ -31,3 +31,13 @@
     </inertial>
   </xacro:macro>
+  <!-- sphere inertial macro with explicit origin parameters -->
+  <xacro:macro name="inertial_sphere" params="mass radius *origin">
+      <inertial>
+          <xacro:insert_block name="origin"/>
+          <mass value="${mass}" />
+          <inertia ixx="${(2/5) * mass * (radius*radius)}" ixy="0.0" ixz="0.0"
+                  iyy="${(2/5) * mass * (radius*radius)}" iyz="0.0"
+                  izz="${(2/5) * mass * (radius*radius)}" />
+      </inertial>
+  </xacro:macro>
 </robot>

File: src/sec_bot/description/robot.urdf.xacro (robot description, xacro)
@@ -1,6 +1,6 @@
 <?xml version="1.0"?>
-<robot xmlns:xacro="http://www.ros.org/wiki/xacro"  name="sec_bot">
+<robot xmlns:xacro="http://www.ros.org/wiki/xacro"  name="robot">
     <xacro:include filename="robot_core.xacro" />
-    <xacro:include filename="gazebo_control.xacro" />
-    <xacro:include filename="camera.xacro" />
+ <!-- <xacro:include filename="gazebo_control.xacro" /> -->
+ <!-- <xacro:include filename="camera.xacro" /> -->
 </robot>

File: src/sec_bot/description/robot_core.xacro (robot description, xacro)
@@ -1,152 +1,201 @@
 <?xml version="1.0"?>
-<robot xmlns:xacro="http://www.ros.org/wiki/xacro" >
-    <xacro:include filename="inertial_macros.xacro"/>
-    <material name="white">
-        <color rgba="1 1 1 1" />
-    </material>
-    <material name="orange">
-        <color rgba="1 0.3 0.1 1"/>
-    </material>
-    <material name="blue">
-        <color rgba="0.2 0.2 1 1"/>
-    </material>
-    <material name="black">
-        <color rgba="0 0 0 1"/>
-    </material>
-    <!-- BASE LINK -->
-    <link name="base_link">
+<robot xmlns:xacro="http://www.ros.org/wiki/xacro" name="robot">
+  <!-- Define ALL materials here -->
+  <material name="white"><color rgba="1 1 1 1"/></material>
+  <material name="blue"><color rgba="0.2 0.2 1 1"/></material>
+  <material name="camera_red"><color rgba="1 0 0 1"/></material>
+  <!-- Includes -->
+  <xacro:include filename="inertial_macros.xacro"/>
+  <!-- Parameters -->
+  <xacro:property name="M_PI" value="3.1415926535897931" />
+  <xacro:property name="left_back_wheel_pos" value="-0.1 0.175 0"/>
+  <xacro:property name="right_back_wheel_pos" value="-0.1 -0.175 0"/>
+  <xacro:property name="left_front_wheel_pos" value="0.1 0.175 0"/>
+  <xacro:property name="right_front_wheel_pos" value="0.1 -0.175 0"/>
+  <!-- Base Structure -->
+  <link name="base_link">
+    <inertial>
+      <mass value="0.001"/>
+      <inertia ixx="0.0001" ixy="0" ixz="0" iyy="0.0001" iyz="0" izz="0.0001"/>
+    </inertial>
+  </link>
+  <joint name="chassis_joint" type="fixed">
+    <parent link="base_link"/>
+    <child link="chassis"/>
+    <origin xyz="0 0 0.05"/>
+  </joint>
+  <link name="chassis">
+    <visual>
+      <origin xyz="0 0 0.125"/>
+      <geometry><box size="0.3 0.3 0.25"/></geometry>
+      <material name="white"/>
+    </visual>
+    <collision>
+      <origin xyz="0 0 0.125"/>
+      <geometry><box size="0.3 0.3 0.25"/></geometry>
+    </collision>
+    <inertial>
+      <mass value="1.0"/>
+      <origin xyz="0 0 0.125"/>
+      <inertia ixx="0.015" ixy="0" ixz="0" iyy="0.0375" iyz="0" izz="0.0375"/>
+    </inertial>
+  </link>
+  <!-- Wheel Macro -->
+  <xacro:macro name="full_wheel" params="name parent origin rpy">
+    <joint name="${name}_joint" type="continuous">
+      <parent link="${parent}"/>
+      <child link="${name}"/>
+      <origin xyz="${origin}" rpy="${rpy}"/>
+      <axis xyz="0 1 0"/>
+    </joint>
+    <link name="${name}">
+      <visual>
+        <geometry><cylinder radius="0.08255" length="0.04"/></geometry>
+        <material name="blue"/>
+      </visual>
+      <collision>
+        <geometry><cylinder radius="0.08255" length="0.04"/></geometry>
+      </collision>
+      <xacro:inertial_cylinder mass="0.1" radius="0.08255" length="0.04"/>
     </link>
-    <!-- CHASSIS LINK -->
-    <joint name="chassis_joint" type="fixed">
-        <parent link="base_link"/>
-        <child link="chassis"/>
-        <origin xyz="-0.1 0 0"/>
-    </joint>
-    <link name="chassis">
-        <visual>
-            <origin xyz="0.19 0 0.125"/>
-            <geometry>
-                <box size="0.3 0.3 0.25"/>
-            </geometry>
-            <material name="white"/>
-        </visual>
-        <collision>
-            <origin xyz="0.19 0 0.125"/>
-            <geometry>
-                <box size="0.3 0.3 0.15"/>
-            </geometry>
-        </collision>
-        <xacro:inertial_box mass="0.5" x="0.3" y="0.3" z="0.15">
-            <origin xyz="0.15 0 0.075" rpy="0 0 0"/>
-        </xacro:inertial_box>
-    </link>
-    <gazebo reference="chassis">
-        <material>Gazebo/White</material>
-    </gazebo>
-    <!-- LEFT BACK WHEEL LINK -->
-    <joint name="left_back_wheel_joint" type="continuous">
-        <parent link="base_link"/>
-        <child link="left_back_wheel"/>
-        <origin xyz="-0.02 0.1400242 0" rpy="-${pi/2} 0 0" />
-        <axis xyz="0 0 1"/>
-    </joint>
-    <link name="left_back_wheel">
-        <visual>
-            <geometry>
-                <cylinder radius="0.08255" length="0.020955"/>
-            </geometry>
-            <material name="blue"/>
-        </visual>
-        <collision>
-            <geometry>
-                <cylinder radius="0.08255" length="0.020955"/>
-            </geometry>
-        </collision>
-        <xacro:inertial_cylinder mass="0.1" length="0.020955" radius="0.08255">
-            <origin xyz="0 0 0" rpy="0 0 0"/>
-        </xacro:inertial_cylinder>
-    </link>
-    <gazebo reference="left_back_wheel">
-        <material>Gazebo/Blue</material>
-    </gazebo>
-    <!-- RIGHT BACK WHEEL LINK -->
-    <joint name="right_back_wheel_joint" type="continuous">
-        <parent link="base_link"/>
-        <child link="right_back_wheel"/>
-        <origin xyz="-0.02 -0.1400242 0" rpy="${pi/2} 0 0" />
-        <axis xyz="0 0 -1"/>
-    </joint>
-    <link name="right_back_wheel">
-        <visual>
-            <geometry>
-                <cylinder radius="0.08255" length="0.020955"/>
-            </geometry>
-            <material name="blue"/>
-        </visual>
-        <collision>
-            <geometry>
-                <cylinder radius="0.08255" length="0.020955"/>
-            </geometry>
-        </collision>
-        <xacro:inertial_cylinder mass="0.1" length="0.020955" radius="0.08255">
-            <origin xyz="0 0 0" rpy="0 0 0"/>
-        </xacro:inertial_cylinder>
-    </link>
-    <gazebo reference="right_back_wheel">
-        <material>Gazebo/Blue</material>
-    </gazebo>
-    <!-- LEFT FRONT WHEEL LINK -->
-    <joint name="left_front_wheel_joint" type="continuous">
-        <parent link="base_link"/>
-        <child link="left_front_wheel"/>
-        <origin xyz="0.2 0.1400242 0" rpy="-${pi/2} 0 0" />
-        <axis xyz="0 0 1"/>
-    </joint>
-    <link name="left_front_wheel">
-        <visual>
-            <geometry>
-                <cylinder radius="0.08255" length="0.020955"/>
-            </geometry>
-            <material name="blue"/>
-        </visual>
-        <collision>
-            <geometry>
-                <cylinder radius="0.08255" length="0.020955"/>
-            </geometry>
-        </collision>
-        <xacro:inertial_cylinder mass="0.1" length="0.020955" radius="0.08255">
-            <origin xyz="0 0 0" rpy="0 0 0"/>
-        </xacro:inertial_cylinder>
-    </link>
-    <gazebo reference="left_front_wheel">
-        <material>Gazebo/Blue</material>
-    </gazebo>
-    <!-- RIGHT FRONT WHEEL LINK -->
-    <joint name="right_front_wheel_joint" type="continuous">
-        <parent link="base_link"/>
-        <child link="right_front_wheel"/>
-        <origin xyz="0.2 -0.1400242 0" rpy="${pi/2} 0 0" />
-        <axis xyz="0 0 -1"/>
-    </joint>
-    <link name="right_front_wheel">
-        <visual>
-            <geometry>
-                <cylinder radius="0.08255" length="0.020955"/>
-            </geometry>
-            <material name="blue"/>
-        </visual>
-        <collision>
-            <geometry>
-                <cylinder radius="0.08255" length="0.020955"/>
-            </geometry>
-        </collision>
-        <xacro:inertial_cylinder mass="0.1" length="0.020955" radius="0.08255">
-            <origin xyz="0 0 0" rpy="0 0 0"/>
-        </xacro:inertial_cylinder>
-    </link>
-    <gazebo reference="right_front_wheel">
-        <material>Gazebo/Blue</material>
-        <mu1 value="0.001"/>
-        <mu2 value="0.001"/>
-    </gazebo>
+    <transmission name="${name}_trans">
+      <type>transmission_interface/SimpleTransmission</type>
+      <joint name="${name}_joint">
+        <hardwareInterface>hardware_interface/VelocityJointInterface</hardwareInterface>
+      </joint>
+      <actuator name="${name}_motor">
+        <mechanicalReduction>1</mechanicalReduction>
+      </actuator>
+    </transmission>
+  </xacro:macro>
+  <!-- Instantiate Wheels -->
+  <xacro:full_wheel name="left_back_wheel" parent="chassis" origin="${left_back_wheel_pos}" rpy="${-(M_PI/2)} 0 0"/>
+  <xacro:full_wheel name="right_back_wheel" parent="chassis" origin="${right_back_wheel_pos}" rpy="${M_PI/2} 0 0"/>
+  <xacro:full_wheel name="left_front_wheel" parent="chassis" origin="${left_front_wheel_pos}" rpy="${-(M_PI/2)} 0 0"/>
+  <xacro:full_wheel name="right_front_wheel" parent="chassis" origin="${right_front_wheel_pos}" rpy="${M_PI/2} 0 0"/>
+  <!-- Gazebo Visuals -->
+  <gazebo reference="chassis">
+    <material>Gazebo/White</material>
+    <mu1>0.2</mu1>
+    <mu2>0.2</mu2>
+    <selfCollide>true</selfCollide>
+  </gazebo>
+  <gazebo reference="left_back_wheel">
+    <material>Gazebo/Blue</material>
+    <mu1>1.0</mu1>
+    <mu2>1.0</mu2>
+    <selfCollide>true</selfCollide>
+  </gazebo>
+  <gazebo reference="right_back_wheel">
+    <material>Gazebo/Blue</material>
+    <mu1>1.0</mu1>
+    <mu2>1.0</mu2>
+    <selfCollide>true</selfCollide>
+  </gazebo>
+  <gazebo reference="left_front_wheel">
+    <material>Gazebo/Blue</material>
+    <mu1>1.0</mu1>
+    <mu2>1.0</mu2>
+    <selfCollide>true</selfCollide>
+  </gazebo>
+  <gazebo reference="right_front_wheel">
+    <material>Gazebo/Blue</material>
+    <mu1>1.0</mu1>
+    <mu2>1.0</mu2>
+    <selfCollide>true</selfCollide>
+  </gazebo>
+  <!-- Cameras -->
+  <!-- Left Camera -->
+  <joint name="camera_joint" type="fixed">
+    <parent link="chassis"/>
+    <child link="camera_link"/>
+    <origin xyz="0.12 0.12 0.25" rpy="0 0 0"/>
+  </joint>
+  <link name="camera_link">
+    <visual>
+      <geometry><box size="0.010 0.03 0.03"/></geometry>
+      <material name="camera_red"/>
+    </visual>
+    <collision>
+      <geometry><box size="0.010 0.03 0.03"/></geometry>
+    </collision>
+    <inertial>
+      <mass value="0.05"/>
+      <inertia ixx="0.0001" ixy="0" ixz="0" iyy="0.0001" iyz="0" izz="0.0001"/>
+    </inertial>
+  </link>
+  <joint name="camera_optical_joint" type="fixed">
+    <parent link="camera_link"/>
+    <child link="camera_link_optical"/>
+    <origin xyz="0 0 0" rpy="${-M_PI/2} 0 ${-M_PI/2}"/>
+  </joint>
+  <link name="camera_link_optical"/>
+  <!-- Right Camera -->
+  <joint name="camera2_joint" type="fixed">
+    <parent link="chassis"/>
+    <child link="camera2_link"/>
+    <origin xyz="0.12 -0.12 0.25" rpy="0 0 0"/>
+  </joint>
+  <link name="camera2_link">
+    <visual>
+      <geometry><box size="0.010 0.03 0.03"/></geometry>
+      <material name="camera_red"/>
+    </visual>
+    <collision>
+      <geometry><box size="0.010 0.03 0.03"/></geometry>
+    </collision>
+    <inertial>
+      <mass value="0.05"/>
+      <inertia ixx="0.0001" ixy="0" ixz="0" iyy="0.0001" iyz="0" izz="0.0001"/>
+    </inertial>
+  </link>
+  <joint name="camera2_optical_joint" type="fixed">
+    <parent link="camera2_link"/>
+    <child link="camera2_link_optical"/>
+    <origin xyz="0 0 0" rpy="${-M_PI/2} 0 ${-M_PI/2}"/>
+  </joint>
+  <link name="camera2_link_optical"/>
+  <!-- Gazebo Harmonic Camera Sensors -->
+  <gazebo reference="camera_link">
+    <material>Gazebo/Red</material>
+    <sensor name="camera_sensor" type="camera">
+      <pose>0 0 0 0 0 0</pose>
+      <update_rate>10</update_rate>
+      <camera>
+        <horizontal_fov>1.089</horizontal_fov>
+        <image>
+          <format>R8G8B8</format>
+          <width>640</width>
+          <height>480</height>
+        </image>
+        <clip>
+          <near>0.05</near>
+          <far>8.0</far>
+        </clip>
+      </camera>
+      <always_on>true</always_on>
+      <visualize>true</visualize>
+    </sensor>
+  </gazebo>
+  <gazebo reference="camera2_link">
+    <material>Gazebo/Red</material>
+    <sensor name="camera2_sensor" type="camera">
+      <pose>0 0 0 0 0 0</pose>
+      <update_rate>10</update_rate>
+      <camera>
+        <horizontal_fov>1.089</horizontal_fov>
+        <image>
+          <format>R8G8B8</format>
+          <width>640</width>
+          <height>480</height>
+        </image>
+        <clip>
+          <near>0.05</near>
+          <far>8.0</far>
+        </clip>
+      </camera>
+      <always_on>true</always_on>
+      <visualize>true</visualize>
+    </sensor>
+  </gazebo>
 </robot>
